Commit message: T Shaped object

File: Gazebo_files/simulation_vvm/urdf/Main_vvm_02.urdf (robot description, URDF)
Before this commit: robot VoiceVidManipulator, 10 links, 9 joints
Links:
- added link horizontal_bar, mass 0.1; visual box size=0.15 0.02 0.05
- added link vertical_bar, mass 0.2; visual box size=0.05 0.05 0.10
Joints:
- added joint fixed_joint: type fixed, parent vertical_bar, child horizontal_bar, origin xyz=0 0.025 0.05
- added joint t_shape_position: type floating, parent world, child vertical_bar, origin xyz=0.280 0 0.078 rpy=0 0 0
