Commit message: joint trajectory and world spawned

File: Gazebo_files/simulation_vvm/urdf/MAIN_vvm.urdf (robot description, URDF)
Before this commit: robot VoiceVidManipulator, 10 links, 9 joints
Links:
- link link5: geometry collision mesh filename=package://simulation_vvm/meshes/chain_link5.stl scale=0.001 0.001 0.001; visual mesh filename=package://simulation_vvm/meshes/chain_link5.stl scale=0.001 0.001 0.001
Joints:
- joint camera_to_camera_frame_joint: origin xyz=0 0 0 rpy=0 -1.5708 0 -> xyz=0.045 0.012 0 rpy=0 1.5708 0

Commit message: added object detection

File: Gazebo_files/simulation_vvm/urdf/MAIN_vvm.urdf (robot description, URDF)
Before this commit: robot VoiceVidManipulator, 10 links, 9 joints
Joints:
- joint camera_to_camera_frame_joint: origin xyz=0.045 0.012 0 rpy=0 1.5708 0 -> xyz=0.045 0.012 0 rpy=0 1.5708 -1.5708
